Commit message: 1

File: capstone/description/face.xacro (robot description, xacro)
@@ -10,5 +10,5 @@
             <origin xyz="0 0.05 0.01" rpy="0 ${pi/2} 0"/>
             <geometry>
-                <cylinder radius="0.02" length="0.003"/>
+                <cylinder radius="0.01" length="0.002"/>
             </geometry>
             <material name="black"/>
@@ -17,5 +17,5 @@
             <origin xyz="0 -0.05 0.01" rpy="0 ${pi/2} 0"/>
             <geometry>
-                <cylinder radius="0.02" length="0.003"/>
+                <cylinder radius="0.01" length="0.002"/>
             </geometry>
             <material name="black"/>
@@ -24,5 +24,5 @@
             <origin xyz="-0.011 0 -0.00" rpy="0 ${1.5} 0"/>
             <geometry>
-                <cylinder radius="0.06" length="0.02"/>
+                <cylinder radius="0.05" length="0.02"/>
             </geometry>
             <material name="red"/>

File: capstone/description/robot_core.xacro (robot description, xacro)
@@ -3,11 +3,11 @@
     <xacro:include filename="inertial_macros.xacro"/>
     <xacro:property name="chassis_length" value="0.335"/>
-    <xacro:property name="chassis_width" value="0.275"/>
-    <xacro:property name="chassis_height" value="0.168"/>
+    <xacro:property name="chassis_width" value="0.265"/>
+    <xacro:property name="chassis_height" value="0.138"/>
     <xacro:property name="chassis_mass" value="1.0"/>
     <xacro:property name="wheel_radius" value="0.038"/>
-    <xacro:property name="wheel_thickness" value="0.029"/>
-    <xacro:property name="wheel_mass" value="0.06"/>
-    <xacro:property name="wheel_offset_x" value="0.206"/>
+    <xacro:property name="wheel_thickness" value="0.026"/>
+    <xacro:property name="wheel_mass" value="0.05"/>
+    <xacro:property name="wheel_offset_x" value="0.226"/>
     <xacro:property name="wheel_offset_y" value="0.1485"/>
     <xacro:property name="wheel_offset_z" value="0.01"/>
