Commit message: 1

File: capstone/description/odometry.xacro (robot description, xacro)
@@ -3,5 +3,5 @@
     <joint name="odom_joint" type="fixed">
         <parent link="chassis"/>
-        <child link="odom"/>
+        <child link="odom_frame"/>
         <origin xyz="0 0 0" rpy="0 0 0"/>
     </joint>

Commit message: 1

File: capstone/description/odometry.xacro (robot description, xacro)
@@ -2,5 +2,5 @@
 <robot xmlns:xacro="http://www.ros.org/wiki/xacro" >
     <joint name="odom_joint" type="fixed">
-        <parent link="chassis"/>
+        <parent link="base_frame"/>
         <child link="odom_frame"/>
         <origin xyz="0 0 0" rpy="0 0 0"/>

Commit message: 1

File: capstone/description/odometry.xacro (robot description, xacro)
@@ -2,5 +2,5 @@
 <robot xmlns:xacro="http://www.ros.org/wiki/xacro" >
     <joint name="odom_joint" type="fixed">
-        <parent link="base_frame"/>
+        <parent link="base_link"/>
         <child link="odom_frame"/>
         <origin xyz="0 0 0" rpy="0 0 0"/>

Commit message: 1

File: capstone/description/odometry.xacro (robot description, xacro)
@@ -3,8 +3,8 @@
     <joint name="odom_joint" type="fixed">
         <parent link="base_link"/>
-        <child link="odom_frame"/>
+        <child link="odom"/>
         <origin xyz="0 0 0" rpy="0 0 0"/>
     </joint>
-    <link name="odom_frame">
+    <link name="odom">
         <visual>
             <geometry>

Commit message: 1

File: capstone/description/odometry.xacro (robot description, xacro)
@@ -2,6 +2,6 @@
 <robot xmlns:xacro="http://www.ros.org/wiki/xacro" >
     <joint name="odom_joint" type="fixed">
-        <parent link="base_link"/>
-        <child link="odom"/>
+        <parent link="odom"/>
+        <child link="base_link"/>
         <origin xyz="0 0 0" rpy="0 0 0"/>
     </joint>

Commit message: 1

File: capstone/description/odometry.xacro (robot description, xacro)
@@ -2,9 +2,9 @@
 <robot xmlns:xacro="http://www.ros.org/wiki/xacro" >
     <joint name="odom_joint" type="fixed">
-        <parent link="odom"/>
-        <child link="base_link"/>
+        <parent link="odom_frame"/>
+        <child link="base_footprint"/>
         <origin xyz="0 0 0" rpy="0 0 0"/>
     </joint>
-    <link name="odom">
+    <link name="odom_frame">
         <visual>
             <geometry>

Commit message: 1

File: capstone/description/odometry.xacro (robot description, xacro)
@@ -2,9 +2,9 @@
 <robot xmlns:xacro="http://www.ros.org/wiki/xacro" >
     <joint name="odom_joint" type="fixed">
-        <parent link="odom_frame"/>
-        <child link="base_footprint"/>
+        <parent link="odom"/>
+        <child link="base_link"/>
         <origin xyz="0 0 0" rpy="0 0 0"/>
     </joint>
-    <link name="odom_frame">
+    <link name="odom">
         <visual>
             <geometry>
